File: SAMD-10.kicad_pcb (KiCad board)
At the start: 4 copper layers, 53.3 x 23 mm, 56 parts, among them J1 10118194-0001LF, J2 Conn_01x14, J3 5031821852, J4 B2B-PH-SM4-TB, J5 NPTC072KFMS-RC, J7 Conn_01x17, J96 MOUNTINGHOLE2.5, J97 MOUNTINGHOLE2.5, Q1 mmbt2222, Q2 mmbt2222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

Commit message: changed board name
Other:
- board text added: "SAMD-10"
- board text removed: "SAM_10"
Changed lines of the file:
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@@
     (1 GND power hide)
     (2 PWR power hide)
-    (31 Bottom signal hide)
+    (31 Bottom signal)
     (32 B.Adhes user hide)
     (33 F.Adhes user hide)
@@
     (35 F.Paste user hide)
     (36 B.SilkS user hide)
-    (37 F.SilkS user)
+    (37 F.SilkS user hide)
     (38 B.Mask user hide)
     (39 F.Mask user hide)
@@
     (effects (font (size 0.635 0.635) (thickness 0.127)))
   )
-  (gr_text SAM_10 (at 83.312 96.393 90) (layer B.SilkS)
+  (gr_text SAMD-10 (at 83.312 96.393 90) (layer B.SilkS)
     (effects (font (size 0.835 0.835) (thickness 0.177)) (justify left mirror))
   )

Commit message: layout DRC
Parts:
- moved C3 0.70 mm to (69.5, 94.2)
Other:
- rule trace_min: 0.127 -> 0.1524
Changed lines of the file:
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@@
     (thickness 1.6)
     (drawings 108)
-    (tracks 1020)
+    (tracks 1019)
     (zones 0)
     (modules 56)
@@
     (zone_clearance 0)
     (zone_45_only no)
-    (trace_min 0.127)
+    (trace_min 0.1524)
     (segment_width 0.1778)
     (edge_width 0.15)
@@
   )
   (module Capacitor_SMD:C_0402_1005Metric (layer Top)
-    (at 68.811 94.234 180)
+    (at 69.5095 94.234 180)
     (descr "Capacitor SMD 0402 (1005 Metric), square (rectangular) end terminal, IPC_7351 nominal, (Body size source: http://www.tortai-tech.com/upload/download/2011102023233369053.pdf), generated with kicad-footprint-generator")
     (tags capacitor)
@@
   (segment (start 70.716 99.672) (end 70.739 99.695) (width 0.381) (layer Top) (net 4))
   (via (at 69.6595 96.647) (size 0.508) (drill 0.254) (layers Top Bottom) (net 4))
-  (segment (start 68.326 94.234) (end 68.326 94.834254) (width 0.2286) (layer Top) (net 4))
-  (via (at 68.339074 94.847328) (size 0.508) (drill 0.254) (layers Top Bottom) (net 4))
-  (segment (start 68.326 94.834254) (end 68.339074 94.847328) (width 0.2286) (layer Top) (net 4))
   (via (at 68.77051 97.409) (size 0.508) (drill 0.254) (layers Top Bottom) (net 4))
   (segment (start 69.6595 95.8595) (end 69.6595 96.647) (width 0.381) (layer Top) (net 4))
@@
   (via (at 102.6795 90.8685) (size 0.508) (drill 0.254) (layers Top Bottom) (net 4))
   (segment (start 102.64256 90.90544) (end 102.6795 90.8685) (width 0.2286) (layer Top) (net 4))
+  (segment (start 69.0245 94.234) (end 69.0245 94.9325) (width 0.2286) (layer Top) (net 4))
+  (via (at 69.0245 94.9325) (size 0.508) (drill 0.254) (layers Top Bottom) (net 4))
   (via (at 72.8345 99.694236) (size 0.508) (drill 0.254) (layers Top Bottom) (net 5))
   (segment (start 72.8345 99.186236) (end 72.8345 99.694236) (width 0.2286) (layer Top) (net 5))
@@
   (segment (start 100.47606 90.90544) (end 100.47606 91.73404) (width 0.2286) (layer Top) (net 5))
   (segment (start 100.47606 91.73404) (end 100.81702 92.075) (width 0.2286) (layer Top) (net 5))
-  (via (at 69.2785 94.9325) (size 0.508) (drill 0.254) (layers Top Bottom) (net 5))
-  (segment (start 69.296 94.234) (end 69.296 94.915) (width 0.2286) (layer Top) (net 5))
-  (segment (start 69.296 94.915) (end 69.2785 94.9325) (width 0.2286) (layer Top) (net 5))
   (via (at 61.9125 94.6785) (size 0.508) (drill 0.254) (layers Top Bottom) (net 5))
   (segment (start 61.918 94.684) (end 61.9125 94.6785) (width 0.1524) (layer Bottom) (net 5))
@@
   (segment (start 62.75294 95.691) (end 62.610015 95.548075) (width 0.2286) (layer Bottom) (net 5))
   (via (at 62.610015 95.548075) (size 0.508) (drill 0.254) (layers Top Bottom) (net 5))
+  (via (at 69.977014 94.9325) (size 0.508) (drill 0.254) (layers Top Bottom) (net 5))
+  (segment (start 69.9945 94.915014) (end 69.977014 94.9325) (width 0.2286) (layer Top) (net 5))
+  (segment (start 69.9945 94.234) (end 69.9945 94.915014) (width 0.2286) (layer Top) (net 5))
   (via (at 97.917004 106.68) (size 0.508) (drill 0.254) (layers Top Bottom) (net 6))
   (segment (start 97.93606 106.699056) (end 97.917004 106.68) (width 0.1524) (layer Top) (net 6))

Commit message: layout review w/ Steve
Routing:
- net IO17: track 14.8 -> 16.6 mm
- net IO39: track 20.6 -> 19.7 mm
- net IO36: track 21.9 -> 21.3 mm
Other:
- board size 53.3 x 23 mm -> 53.4 x 23.4 mm
- board text added: "CHRG"
- board text added: "RED"
- board text added: "SAM32"
- board text added: "uSD"
- board text added: "v10"
- board text removed: "SAMD-10"
- board text removed: "SPI"
