File: SAMD-10.sch (KiCad schematic (older format))
At the start: 56 parts, among them J1 10118194-0001LF, J2 Conn_01x14, J3 5031821852, J4 B2B-PH-SM4-TB, J5 NPTC072KFMS-RC, J7 Conn_01x17, J96 MOUNTINGHOLE2.5, J97 MOUNTINGHOLE2.5, Q1 mmbt2222, Q2 mmbt2222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

Commit message: changed board name
Other:
- note added: "SAMD-10"
- note removed: "SAM32-10"
Changed lines of the file:
@@
 	3400 1100 3400 1650
 Text Notes 7450 7500 0    79   ~ 16
-SAM32-10
+SAMD-10
 Text Notes 8100 6950 0    79   ~ 16
 SAMD51 +ESP32-WROOM + microSD

Commit message: layout review w/ Steve
Parts:
- C1, C10, C11, C13, C14, C15, C3, C5, C8, C9: symbol lab64_SAM32-rescue:CAP_CERAMIC0603_NO-Adafruit_Feather_M4_Express-eagle-import -> SAMD-10-rescue:CAP_CERAMIC0603_NO-Adafruit_Feather_M4_Express-eagle-import-lab64_SAM32-rescue
- C12, C2, C4, C6, C7: symbol lab64_SAM32-rescue:CAP_CERAMIC0805-NOOUTLINE-Adafruit_Feather_M4_Express-eagle-import -> SAMD-10-rescue:CAP_CERAMIC0805-NOOUTLINE-Adafruit_Feather_M4_Express-eagle-import-lab64_SAM32-rescue
- CHRG1, RED1: symbol lab64_SAM32-rescue:LED0805_NOOUTLINE-Adafruit_Feather_M4_Express-eagle-import -> SAMD-10-rescue:LED0805_NOOUTLINE-Adafruit_Feather_M4_Express-eagle-import-lab64_SAM32-rescue
- D1: symbol lab64_SAM32-rescue:DIODE-SCHOTTKYSOD-123-Adafruit_Feather_M4_Express-eagle-import -> SAMD-10-rescue:DIODE-SCHOTTKYSOD-123-Adafruit_Feather_M4_Express-eagle-import-lab64_SAM32-rescue
- J3: symbol lab64_SAM32-rescue:503182-1853-503182-1853-lab64_SAM32-rescue -> SAMD-10-rescue:503182-1853-503182-1853-lab64_SAM32-rescue-lab64_SAM32-rescue
- J4: symbol Adafruit_Feather_M0_Adalogger-eagle-import:CON_JST_PH_2PINSH2 -> SAMD-10-rescue:CON_JST_PH_2PINSH2-Adafruit_Feather_M0_Adalogger-eagle-import
- J5: symbol SMD_Headers:NPPC_0.100in_2ROW -> SAMD-10-rescue:NPPC_0.100in_2ROW-SMD_Headers
- J96, J97: symbol Adafruit_HUZZAH32_ESP32_Feather-eagle-import:MOUNTINGHOLE2.5 -> SAMD-10-rescue:MOUNTINGHOLE2.5-Adafruit_HUZZAH32_ESP32_Feather-eagle-import
- L1: symbol lab64_SAM32-rescue:INDUCTOR-Adafruit_Feather_M4_Express-eagle-import -> SAMD-10-rescue:INDUCTOR-Adafruit_Feather_M4_Express-eagle-import-lab64_SAM32-rescue
- Q1, Q2: symbol lab64_SAM32-rescue:TRANSISTOR_NPNSOT23-3-Adafruit_HUZZAH32_ESP32_Feather-eagle-import -> SAMD-10-rescue:TRANSISTOR_NPNSOT23-3-Adafruit_HUZZAH32_ESP32_Feather-eagle-import-lab64_SAM32-rescue
- Q3: symbol lab64_SAM32-rescue:MOSFET-P-Adafruit_Feather_M4_Express-eagle-import -> SAMD-10-rescue:MOSFET-P-Adafruit_Feather_M4_Express-eagle-import-lab64_SAM32-rescue
- SW1: symbol lab64_SAM32-rescue:SWITCH_TACT_SMT4.6X2.8-Adafruit_Feather_M4_Express-eagle-import -> SAMD-10-rescue:SWITCH_TACT_SMT4.6X2.8-Adafruit_Feather_M4_Express-eagle-import-lab64_SAM32-rescue
- TP1, TP2: symbol Adafruit_Feather_M4_Express-eagle-import:TESTPOINTPAD2MM -> SAMD-10-rescue:TESTPOINTPAD2MM-Adafruit_Feather_M4_Express-eagle-import
- U1: symbol lab64_SAM32-rescue:MAX3202EETT+T-symbols-lab64_SAM32-rescue -> SAMD-10-rescue:MAX3202EETT+T-symbols-lab64_SAM32-rescue-lab64_SAM32-rescue
- U2: symbol lab64_SAM32-rescue:ATSAMD51J20A-AU-ATSAMD51J20A-AU-lab64_SAM32-rescue -> SAMD-10-rescue:ATSAMD51J20A-AU-ATSAMD51J20A-AU-lab64_SAM32-rescue-lab64_SAM32-rescue
- U3: symbol Adafruit_HUZZAH32_ESP32_Feather-eagle-import:ESP32_WROOM32_SKINNY -> SAMD-10-rescue:ESP32_WROOM32_SKINNY-Adafruit_HUZZAH32_ESP32_Feather-eagle-import
- U4: symbol lab64_SAM32-rescue:MCP73831_2-Adafruit_Feather_M4_Express-eagle-import -> SAMD-10-rescue:MCP73831_2-Adafruit_Feather_M4_Express-eagle-import-lab64_SAM32-rescue
- U5: symbol lab64_SAM32-rescue:VREG_SOT23-5-Adafruit_Feather_M4_Express-eagle-import -> SAMD-10-rescue:VREG_SOT23-5-Adafruit_Feather_M4_Express-eagle-import-lab64_SAM32-rescue
Other:
- note added: "SAM32"
- note removed: "SAMD-10"
