File: hardware/SAM32.sch (KiCad schematic (older format))
At the start: 56 parts, among them J1 10118194-0001LF, J2 Conn_01x14, J3 5031821852, J4 B2B-PH-SM4-TB, J5 NPTC072KFMS-RC, J7 Conn_01x17, J96 MOUNTINGHOLE2.5, J97 MOUNTINGHOLE2.5, Q1 mmbt2222, Q2 mmbt2222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

Commit message: updating hardware to v2
Parts:
- removed Q1, Q2: mmbt2222, Adafruit HUZZAH32 ESP32 Feather:SOT23-3, symbol SAMD-10-rescue:TRANSISTOR_NPNSOT23-3-Adafruit_HUZZAH32_ESP32_Feather-eagle-impo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
- removed R1: 100K, Resistors_SMD:R_0402, symbol Device:R_US
- removed R13, R14: 0, Resistors_SMD:R_0402, symbol Device:R_US
- removed RED1: RED LED, LED_SMD:LED_0805_2012Metric, symbol SAMD-10-rescue:LED0805_NOOUTLINE-Adafruit_Feather_M4_Express-eagle-import-lab64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
- added D2: WS2812B, LED_SMD:LED_WS2812B_PLCC4_5.0x5.0mm_P3.2mm, symbol LED:WS2812B
- added GRN1: GREEN LED, LED_SMD:LED_0603_1608Metric, symbol SAM32-rescue:LED0805_NOOUTLINE-Adafruit_Feather_M4_Express-eagle-import-lab64_S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
- C1, C10, C11, C13, C14, C15, C3, C5, C8, C9: symbol SAMD-10-rescue:CAP_CERAMIC0603_NO-Adafruit_Feather_M4_Express-eagle-import-lab64_SAM32-rescue -> SAM32-rescue:CAP_CERAMIC0603_NO-Adafruit_Feather_M4_Express-eagle-import-lab64_SAM32-rescue-SAMD-10-rescue
- C12, C2, C4, C6, C7: footprint Capacitor_SMD:C_0603_1608Metric -> Capacitor_SMD:C_0402_1005Metric; symbol SAMD-10-rescue:CAP_CERAMIC0805-NOOUTLINE-Adafruit_Feather_M4_Express-eagle-import-lab64_SAM32-rescue -> SAM32-rescue:CAP_CERAMIC0805-NOOUTLINE-Adafruit_Feather_M4_Express-eagle-import-lab64_SAM32-rescue-SAMD-10-rescue
- CHRG1: footprint LED_SMD:LED_0805_2012Metric -> LED_SMD:LED_0402_1005Metric; symbol SAMD-10-rescue:LED0805_NOOUTLINE-Adafruit_Feather_M4_Express-eagle-import-lab64_SAM32-rescue -> SAM32-rescue:LED0805_NOOUTLINE-Adafruit_Feather_M4_Express-eagle-import-lab64_SAM32-rescue-SAMD-10-rescue
- D1: symbol SAMD-10-rescue:DIODE-SCHOTTKYSOD-123-Adafruit_Feather_M4_Express-eagle-import-lab64_SAM32-rescue -> SAM32-rescue:DIODE-SCHOTTKYSOD-123-Adafruit_Feather_M4_Express-eagle-import-lab64_SAM32-rescue-SAMD-10-rescue
- J3: symbol SAMD-10-rescue:503182-1853-503182-1853-lab64_SAM32-rescue-lab64_SAM32-rescue -> SAM32-rescue:503182-1853-503182-1853-lab64_SAM32-rescue-lab64_SAM32-rescue-SAMD-10-rescue
- J4: footprint Connector_JST:JST_PH_B2B-PH-SM4-TB_1x02-1MP_P2.00mm_Vertical -> Connector_JST:JST_PH_S2B-PH-SM4-TB_1x02-1MP_P2.00mm_Horizontal; symbol SAMD-10-rescue:CON_JST_PH_2PINSH2-Adafruit_Feather_M0_Adalogger-eagle-import -> SAM32-rescue:CON_JST_PH_2PINSH2-Adafruit_Feather_M0_Adalogger-eagle-import-SAMD-10-rescue
- J5: symbol SAMD-10-rescue:NPPC_0.100in_2ROW-SMD_Headers -> SAM32-rescue:NPPC_0.100in_2ROW-SMD_Headers-SAMD-10-rescue
- J96, J97: symbol SAMD-10-rescue:MOUNTINGHOLE2.5-Adafruit_HUZZAH32_ESP32_Feather-eagle-import -> SAM32-rescue:MOUNTINGHOLE2.5-Adafruit_HUZZAH32_ESP32_Feather-eagle-import-SAMD-10-rescue
- L1: symbol SAMD-10-rescue:INDUCTOR-Adafruit_Feather_M4_Express-eagle-import-lab64_SAM32-rescue -> SAM32-rescue:INDUCTOR-Adafruit_Feather_M4_Express-eagle-import-lab64_SAM32-rescue-SAMD-10-rescue
- Q3: symbol SAMD-10-rescue:MOSFET-P-Adafruit_Feather_M4_Express-eagle-import-lab64_SAM32-rescue -> SAM32-rescue:MOSFET-P-Adafruit_Feather_M4_Express-eagle-import-lab64_SAM32-rescue-SAMD-10-rescue
- R2: footprint Resistors_SMD:R_0402 -> Resistor_SMD:R_0402_1005Metric
- R3: footprint Resistor_SMD:R_0402 -> Resistor_SMD:R_0402_1005Metric
- R4: footprint Resistor_SMD:R_0603_1608Metric_Pad1.05x0.95mm_HandSolder -> Resistor_SMD:R_0402_1005Metric
- SW1: symbol SAMD-10-rescue:SWITCH_TACT_SMT4.6X2.8-Adafruit_Feather_M4_Express-eagle-import-lab64_SAM32-rescue -> SAM32-rescue:SWITCH_TACT_SMT4.6X2.8-Adafruit_Feather_M4_Express-eagle-import-lab64_SAM32-rescue-SAMD-10-rescue
- TP1, TP2: symbol SAMD-10-rescue:TESTPOINTPAD2MM-Adafruit_Feather_M4_Express-eagle-import -> SAM32-rescue:TESTPOINTPAD2MM-Adafruit_Feather_M4_Express-eagle-import-SAMD-10-rescue
- U1: symbol SAMD-10-rescue:MAX3202EETT+T-symbols-lab64_SAM32-rescue-lab64_SAM32-rescue -> SAM32-rescue:MAX3202EETT+T-symbols-lab64_SAM32-rescue-lab64_SAM32-rescue-SAMD-10-rescue
- U2: symbol SAMD-10-rescue:ATSAMD51J20A-AU-ATSAMD51J20A-AU-lab64_SAM32-rescue-lab64_SAM32-rescue -> SAM32-rescue:ATSAMD51J20A-AU-ATSAMD51J20A-AU-lab64_SAM32-rescue-lab64_SAM32-rescue-SAMD-10-rescue
- U3: symbol SAMD-10-rescue:ESP32_WROOM32_SKINNY-Adafruit_HUZZAH32_ESP32_Feather-eagle-import -> SAM32-rescue:ESP32_WROOM32_SKINNY-Adafruit_HUZZAH32_ESP32_Feather-eagle-import-SAMD-10-rescue
- U4: symbol SAMD-10-rescue:MCP73831_2-Adafruit_Feather_M4_Express-eagle-import-lab64_SAM32-rescue -> SAM32-rescue:MCP73831_2-Adafruit_Feather_M4_Express-eagle-import-lab64_SAM32-rescue-SAMD-10-rescue
- U5: symbol SAMD-10-rescue:VREG_SOT23-5-Adafruit_Feather_M4_Express-eagle-import-lab64_SAM32-rescue -> SAM32-rescue:VREG_SOT23-5-Adafruit_Feather_M4_Express-eagle-import-lab64_SAM32-rescue-SAMD-10-rescue
Connections:
- net MISO: now also U2.27 (PB14); no longer U2.26 (PB13)
- net SCK: now also U2.26 (PB13); no longer U2.27 (PB14)
- net at R2.1: now also GRN1.1
- net at U3.25 (IO0/A2_1): now also R11.2
- net at U3.3 (EN): now also R12.2
- net D32 renamed NEOPIXEL
- net NEOPIXEL: now also D2.4 (DIN)
- net RX: no longer names the net of U3.34 (RXD0)
- net RX: now also U2.39 (PB16); no longer U2.40 (PB17)
- net TX: no longer names the net of U3.35 (TXD0)
- net TX: now also U2.40 (PB17); no longer U2.39 (PB16)
Other:
- note added: "2"
- note added: "MISO"
- note removed: "1"
- moved on the sheet: R11
