File: hardware/SAM32.sch (KiCad schematic (older format))
At the start: 52 parts, among them J1 10118194-0001LF, J2 Conn_01x14, J3 5031821852, J4 B2B-PH-SM4-TB, J5 NPTC072KFMS-RC, J7 Conn_01x17, J96 MOUNTINGHOLE2.5, J97 MOUNTINGHOLE2.5, Q3 DMG341, SW1 KMR231NG LFS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

Commit message: updating more documention to v2a
Parts:
- removed D1: MBR120, Adafruit Feather M4 Express:SOD-123, symbol SAM32-rescue:DIODE-SCHOTTKYSOD-123-Adafruit_Feather_M4_Express-eagle-import-lab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
- added D1: MBR120, Diode_SMD:D_SC-80, symbol Device:D
- added R1: 10K, Resistors_SMD:R_0402, symbol Device:R_US
- D2: footprint LED_SMD:LED_WS2812B_PLCC4_5.0x5.0mm_P3.2mm -> custom-footprints:LED3535
- U1: DNI (none) -> DNI
Connections:
- net labels added: ~RTS
- net labels removed: NEOPIXEL, RTS
- wire segments 256 -> 247
Other:
- note added: "2.1"
- note added: "Hold DTR low during boot\nfor serial bootloader access"
- note added: "NEOPIXEL"
- note removed: "2"
- note removed: "ESP32 AUTORESET"
- note removed: "MISO"
- moved on the sheet: D2, R15, R16, R17, R3, R5

Commit message: unifying footprints
Parts:
- R1, R11, R12, R15, R16, R17, R9: footprint Resistors_SMD:R_0402 -> Resistor_SMD:R_0402_1005Metric
- R10, R5, R6, R7, R8: footprint Resistor_SMD:R_0402 -> Resistor_SMD:R_0402_1005Metric
Changed lines of the file:
@@
 U 1 1 5C02C9DB
 P 1700 2750
-F 0 "R3" H 1550 2650 50  0000 C CNN
+F 0 "R3" H 1800 2850 50  0000 C CNN
 F 1 "100K" H 1850 2750 50  0000 C CNN
 F 2 "Resistor_SMD:R_0402_1005Metric" V 1740 2740 50  0001 C CNN
@@
 F 0 "R10" H 2750 1400 50  0000 C CNN
 F 1 "10K" H 2750 1300 50  0000 C CNN
-F 2 "Resistor_SMD:R_0402" V 2690 1340 50  0001 C CNN
+F 2 "Resistor_SMD:R_0402_1005Metric" V 2690 1340 50  0001 C CNN
 F 3 "~" H 2650 1350 50  0001 C CNN
 	1    2650 1350
@@
 F 0 "R7" H 8000 1700 50  0000 C CNN
 F 1 "1K" H 8000 1600 50  0000 C CNN
-F 2 "Resistor_SMD:R_0402" V 8190 1640 50  0001 C CNN
+F 2 "Resistor_SMD:R_0402_1005Metric" V 8190 1640 50  0001 C CNN
 F 3 "~" H 8150 1650 50  0001 C CNN
 	1    8150 1650
@@
 F 0 "R6" H 9350 1750 50  0000 C CNN
 F 1 "10K" H 9300 1350 50  0000 C CNN
-F 2 "Resistor_SMD:R_0402" V 9390 1540 50  0001 C CNN
+F 2 "Resistor_SMD:R_0402_1005Metric" V 9390 1540 50  0001 C CNN
 F 3 "~" H 9350 1550 50  0001 C CNN
 	1    9350 1550
@@
 F 0 "R9" H 2300 1400 50  0000 C CNN
 F 1 "10K" H 2300 1300 50  0000 C CNN
-F 2 "Resistors_SMD:R_0402" V 2490 1340 50  0001 C CNN
+F 2 "Resistor_SMD:R_0402_1005Metric" V 2490 1340 50  0001 C CNN
 F 3 "~" H 2450 1350 50  0001 C CNN
 	1    2450 1350
@@
 U 1 1 5C08F158
 P 1550 2900
-F 0 "R5" V 1250 3150 50  0000 C CNN
+F 0 "R5" V 1450 2900 50  0000 C CNN
 F 1 "100K" V 1650 2900 50  0000 C CNN
-F 2 "Resistor_SMD:R_0402" V 1590 2890 50  0001 C CNN
+F 2 "Resistor_SMD:R_0402_1005Metric" V 1590 2890 50  0001 C CNN
 F 3 "~" H 1550 2900 50  0001 C CNN
 	1    1550 2900
@@
 F 0 "R15" V 7400 4500 50  0000 C CNN
 F 1 "0" V 7400 4750 50  0000 C CNN
-F 2 "Resistors_SMD:R_0402" V 7490 4640 50  0001 C CNN
+F 2 "Resistor_SMD:R_0402_1005Metric" V 7490 4640 50  0001 C CNN
 F 3 "~" H 7450 4650 50  0001 C CNN
 	1    7450 4650
@@
 F 0 "R16" V 7400 4600 50  0000 C CNN
 F 1 "0" V 7400 4850 50  0000 C CNN
-F 2 "Resistors_SMD:R_0402" V 7490 4740 50  0001 C CNN
+F 2 "Resistor_SMD:R_0402_1005Metric" V 7490 4740 50  0001 C CNN
 F 3 "~" H 7450 4750 50  0001 C CNN
 	1    7450 4750
@@
 F 0 "R17" V 7400 4700 50  0000 C CNN
 F 1 "0" V 7400 4950 50  0000 C CNN
-F 2 "Resistors_SMD:R_0402" V 7490 4840 50  0001 C CNN
+F 2 "Resistor_SMD:R_0402_1005Metric" V 7490 4840 50  0001 C CNN
 F 3 "~" H 7450 4850 50  0001 C CNN
 	1    7450 4850
@@
 F 0 "R11" V 5850 3550 50  0000 C CNN
 F 1 "10K" V 5850 3200 50  0000 C CNN
-F 2 "Resistors_SMD:R_0402" V 5840 3390 50  0001 C CNN
+F 2 "Resistor_SMD:R_0402_1005Metric" V 5840 3390 50  0001 C CNN
 F 3 "~" H 5800 3400 50  0001 C CNN
 	1    5800 3400
@@
 F 0 "R12" V 5850 3650 50  0000 C CNN
 F 1 "10K" V 5850 3300 50  0000 C CNN
-F 2 "Resistors_SMD:R_0402" V 5840 3490 50  0001 C CNN
+F 2 "Resistor_SMD:R_0402_1005Metric" V 5840 3490 50  0001 C CNN
 F 3 "~" H 5800 3500 50  0001 C CNN
 	1    5800 3500
@@
 F 0 "R8" H 1750 5350 50  0000 C CNN
 F 1 "1M" H 1750 5450 50  0000 C CNN
-F 2 "Resistor_SMD:R_0402" V 1690 5390 50  0001 C CNN
+F 2 "Resistor_SMD:R_0402_1005Metric" V 1690 5390 50  0001 C CNN
 F 3 "~" H 1650 5400 50  0001 C CNN
 	1    1650 5400
@@
 F 0 "R1" H 4750 4350 50  0000 C CNN
 F 1 "10K" H 4750 4250 50  0000 C CNN
-F 2 "Resistors_SMD:R_0402" V 4940 4290 50  0001 C CNN
+F 2 "Resistor_SMD:R_0402_1005Metric" V 4940 4290 50  0001 C CNN
 F 3 "~" H 4900 4300 50  0001 C CNN
 	1    4900 4300

Commit message: modified board pinout to conform to adafruit feather standard :+1:
Parts:
- added R13, R14: 10K, Resistor_SMD:R_0402_1005Metric, symbol Device:R_US
Connections:
- net labels added: D16, RX, TX, VIN
- net labels removed: AIN2, AIN3, D29, D30
- wire segments 247 -> 256
Other:
- moved on the sheet: R15, R16, R17
