File: hardware/SAM32.kicad_pcb (KiCad board)
At the start: 4 copper layers, 53.4 x 23.4 mm, 56 parts, among them J1 10118194-0001LF, J2 Conn_01x14, J3 5031821852, J4 B2B-PH-SM4-TB, J5 NPTC072KFMS-RC, J7 Conn_01x17, J96 MOUNTINGHOLE2.5, J97 MOUNTINGHOLE2.5, Q1 mmbt2222, Q2 mmbt2222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

Commit message: updating hardware to v2
Parts:
- removed Q1, Q2: mmbt2222, Adafruit HUZZAH32 ESP32 Feather:SOT23-3
- removed R1: 100K, Resistors_SMD:R_0402
- removed R13, R14: 0, Resistors_SMD:R_0402
- removed RED1: RED LED, LED_SMD:LED_0805_2012Metric
- added D2: WS2812B, LED_SMD:LED_WS2812B_PLCC4_5.0x5.0mm_P3.2mm, F.Cu at (63.6, 105.3)
- added GRN1: GREEN LED, LED_SMD:LED_0603_1608Metric, F.Cu at (59.0, 93.4)
- C12, C2, C4, C6, C7: footprint Capacitor_SMD:C_0603_1608Metric -> Capacitor_SMD:C_0402_1005Metric
- CHRG1: footprint LED_SMD:LED_0805_2012Metric -> LED_SMD:LED_0402_1005Metric
- J4: footprint Connector_JST:JST_PH_B2B-PH-SM4-TB_1x02-1MP_P2.00mm_Vertical -> Connector_JST:JST_PH_S2B-PH-SM4-TB_1x02-1MP_P2.00mm_Horizontal
- R2: footprint Resistors_SMD:R_0402 -> Resistor_SMD:R_0402_1005Metric; moved to B.Cu
- R3: footprint Resistor_SMD:R_0402 -> Resistor_SMD:R_0402_1005Metric
- R4: footprint Resistor_SMD:R_0603_1608Metric_Pad1.05x0.95mm_HandSolder -> Resistor_SMD:R_0402_1005Metric
- moved C9 11.8 mm to (63.7, 94.2), turned to 180 degrees
- moved SW1 6.01 mm to (63.5, 99.5), turned to 270 degrees
- moved R2 5.52 mm to (61.6, 92.8), turned to 0 degrees
- moved R12 3.01 mm to (78.5, 104.4), turned to 0 degrees
- moved R3 2.92 mm to (71.5, 100.1)
- moved R11 2.91 mm to (78.5, 105.9), turned to 0 degrees
- moved C5 1.76 mm to (71.7, 99.1), turned to 0 degrees
- moved C1 1.36 mm to (67.9, 97.0), turned to 180 degrees
- moved D1 1.26 mm to (67.8, 98.8)
- moved C7 1.19 mm to (68.5, 104.0), turned to 180 degrees
- moved Q3 1.16 mm to (67.8, 101.1)
- moved C6 1.02 mm to (73.2, 99.4), turned to 270 degrees
- moved R9 0.95 mm to (61.7, 94.2), turned to 0 degrees
- moved C3 0.69 mm to (70.2, 94.1)
- moved CHRG1 0.68 mm to (70.1, 104.5)
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Connections:
- R11 pad 2: Net-(Q1-Pad1) -> Net-(R11-Pad2)
- R12 pad 2: Net-(Q2-Pad1) -> Net-(R12-Pad2)
- U2 pad 26: MISO -> SCK
- U2 pad 27: SCK -> MISO
- U2 pad 32: D32 -> NEOPIXEL
- U2 pad 39: /TX -> Net-(U2-Pad39)
- U2 pad 40: /RX -> Net-(U2-Pad40)
- U3 pad 25: Net-(R14-Pad1) -> Net-(R11-Pad2)
- U3 pad 3: Net-(R13-Pad1) -> Net-(R12-Pad2)
- U3 pad 34: /RX -> Net-(U2-Pad39)
- U3 pad 35: /TX -> Net-(U2-Pad40)
Routing:
- net Net-(U2-Pad40): track 0.00 -> 39.1 mm, vias 0 -> 1
- net /TX: track 39.0 -> 0.00 mm, vias 1 -> 0
- net /RX: track 39.0 -> 0.00 mm, vias 1 -> 0
- net Net-(U2-Pad39): track 0.00 -> 37.9 mm, vias 0 -> 1
- net Net-(R12-Pad2): track 0.00 -> 36.5 mm, vias 0 -> 1
- net Net-(R13-Pad1): track 32.9 -> 0.00 mm, vias 1 -> 0
- net /~RESET: track 28.9 -> 16.7 mm
- net Net-(R11-Pad2): track 0.00 -> 8.72 mm, vias 0 -> 1
- net /DTR: track 16.7 -> 9.50 mm
- net VUSB: track 29.7 -> 25.0 mm
- net Net-(Q2-Pad3): track 4.60 -> 0.00 mm
- net Net-(Q2-Pad1): track 3.97 -> 0.00 mm
- net Net-(Q1-Pad1): track 3.86 -> 0.00 mm
- net Net-(Q1-Pad3): track 3.73 -> 0.00 mm
- net D35: track 27.1 -> 23.7 mm
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Other:
- outline, holes or cut-outs redrawn
- rule trace_min: 0.1524 -> 0.127
- rule via_min_size: 0.508 -> 0.254
- board text added: "GRN"
- board text added: "HOLLIDAY"
- board text added: "IO 26"
- board text added: "RST"
- board text added: "VBAT"
- board text added: "v20"
- board text removed: "BOTTOM"
- board text removed: "IO26"
- board text removed: "LYR1"
- board text removed: "LYR2"
- board text removed: "LYR3"
- board text removed: "LYR4"
- board text removed: "RED"
- board text removed: "RESET"
- board text removed: "TOP"
- board text removed: "v10"

Commit message: updating more documention to v2a
Parts:
- added R1: 10K, Resistors_SMD:R_0402, B.Cu at (78.5, 103.5)
- D1: footprint Adafruit Feather M4 Express:SOD-123 -> Diode_SMD:D_SC-80
- D2: footprint LED_SMD:LED_WS2812B_PLCC4_5.0x5.0mm_P3.2mm -> custom-footprints:LED3535
- moved D2 0.96 mm to (63.8, 104.4)
- moved SW1 0.70 mm to (64.2, 99.8)
- moved GRN1 0.36 mm to (59.0, 93.8)
- moved R12 0.28 mm to (78.5, 104.7)
- moved D1 0.18 mm to (67.6, 98.7)
Connections:
- net /RTS renamed /~RTS
- net NEOPIXEL renamed Net-(D2-Pad4)
Routing:
- net GND: track 30.6 -> 33.2 mm
- net /~RESET: track 16.7 -> 15.3 mm
- net Net-(R1-Pad2): track 37.9 -> 39.1 mm
- net VUSB: track 25.0 -> 26.1 mm
- net Net-(D2-Pad4): track 2.27 -> 2.83 mm
- net +3V3: track 18.9 -> 19.2 mm, vias 17 -> 18
Other:
- board text added: "LED"
- board text added: "v21"
- board text removed: "GRN"
- board text removed: "v20"

Commit message: unifying footprints
Parts:
- R1, R11, R12, R15, R16, R17, R9: footprint Resistors_SMD:R_0402 -> Resistor_SMD:R_0402_1005Metric
- R10, R5, R6, R7, R8: footprint Resistor_SMD:R_0402 -> Resistor_SMD:R_0402_1005Metric
