File: hardware/SAM32_v22/SAM32.kicad_pcb (KiCad board)
At the start: 4 copper layers, 53.4 x 23.4 mm, 55 parts, among them J1 10118194-0001LF, J2 Conn_01x14, J3 5031821852, J4 B2B-PH-SM4-TB, J5 NPTC072KFMS-RC, J7 Conn_01x17, J96 MOUNTINGHOLE2.5, J97 MOUNTINGHOLE2.5, Q3 DMG341, SW1 KMR231NG LFS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

Commit message: v22 cleanup and output files
Parts:
- removed U1: MAX3202EETT+T, custom-footprints:WLP-4-0.5
- moved C14 0.07 mm to (79.7, 97.7)
Connections:
- net /TCK renamed TCK
- net /TDI renamed TDI
- net /TMS renamed TMS
- J7 pad 3: D42 -> D43
- J7 pad 5: D43 -> D42
- J7 pad 6: Net-(J7-Pad6) -> D41
Routing:
- net D41: track 0.00 -> 21.9 mm, vias 0 -> 1
- net VUSB: track 26.0 -> 20.2 mm, vias 1 -> 0
- net D42: track 14.8 -> 20.6 mm
- net D43: track 21.8 -> 16.5 mm, vias 1 -> 0
- net /USB+: track 8.33 -> 5.71 mm
- net +3V3: track 18.0 -> 19.0 mm
- net /USB-: track 6.50 -> 5.72 mm
- net SCK: track 43.3 -> 44.0 mm
- net GND: track 30.7 -> 30.0 mm, vias 40 -> 39
Other:
- board text added: "D41"
- board text added: "v22"
- board text removed: "AIN0"
- board text removed: "AIN1"
- board text removed: "D29"
- board text removed: "D30"
- board text removed: "v21"

Commit message: minor v2.2 fab tweaks
Parts:
- added REF**: Fiducial_0.5mm_Dia_1mm_Outer, Fiducial:Fiducial_0.5mm_Dia_1mm_Outer, B.Cu at (64.7, 89.8)
- added REF**: Fiducial_0.5mm_Dia_1mm_Outer, Fiducial:Fiducial_0.5mm_Dia_1mm_Outer, F.Cu at (64.7, 89.8)
- added REF**: Fiducial_0.5mm_Dia_1mm_Outer, Fiducial:Fiducial_0.5mm_Dia_1mm_Outer, B.Cu at (60.7, 110.0)
- added REF**: Fiducial_0.5mm_Dia_1mm_Outer, Fiducial:Fiducial_0.5mm_Dia_1mm_Outer, F.Cu at (60.7, 110.0)
- added REF**: Fiducial_0.5mm_Dia_1mm_Outer, Fiducial:Fiducial_0.5mm_Dia_1mm_Outer, B.Cu at (104.6, 88.6)
- added REF**: Fiducial_0.5mm_Dia_1mm_Outer, Fiducial:Fiducial_0.5mm_Dia_1mm_Outer, F.Cu at (104.6, 88.6)
- moved D2 0.31 mm to (63.8, 104.7)
- moved C10 0.14 mm to (63.3, 105.1)
