File: hardware/SAM32_v23/SAM32.kicad_pcb (KiCad board)
At the start: 4 copper layers, 53.4 x 23.4 mm, 54 parts, among them J1 10118194-0001LF, J2 Conn_01x14, J3 5031821852, J4 B2B-PH-SM4-TB, J5 NPTC072KFMS-RC, J7 Conn_01x17, J96 MOUNTINGHOLE2.5, J97 MOUNTINGHOLE2.5, Q3 DMG341, SW1 KMR231NG LFS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

Commit message: making v23 easier to clone and work on locally
Parts:
- Q3: footprint Adafruit Feather M4 Express:SOT23-R -> Package_TO_SOT_SMD:SOT-23
- U4, U5: footprint Adafruit Feather M4 Express:SOT23-5 -> Package_TO_SOT_SMD:SOT-23-5
- turned Q3 to 90 degrees
- turned U4 to 0 degrees
- turned U5 to 180 degrees
Connections:
- R11 pad 1: /~RTS -> /DTR
- R12 pad 1: /DTR -> /~RTS
- U2 pad 23: /~RTS -> /DTR
- U2 pad 24: /DTR -> /~RTS
Routing:
- net /~RTS: track 10.3 -> 9.51 mm
- net /DTR: track 9.51 -> 10.3 mm
